Commit message: Fixed wheels urdf

File: jaime_vs/description/gazebo_control.xacro (robot description, xacro)
@@ -6,6 +6,6 @@
             <left_joint>left_wheel_joint</left_joint>
             <right_joint>right_wheel_joint</right_joint>
-            <wheel_separation>0.35</wheel_separation>
-            <wheel_diameter>0.1</wheel_diameter>
+            <wheel_separation>0.23</wheel_separation>
+            <wheel_diameter>0.07</wheel_diameter>
             <!-- Limits -->
             <max_wheel_torque>200</max_wheel_torque>

File: jaime_vs/description/robot_core.xacro (robot description, xacro)
@@ -83,5 +83,5 @@
         <child link="left_wheel"/>
         <origin xyz="0 0.115 -0.025" rpy="-${pi/2} 0 0" />
-        <axis xyz="1 0 0"/>
+        <axis xyz="0 0 1"/>
     </joint>
     <link name="left_wheel">
@@ -98,6 +98,6 @@
             </geometry>
         </collision>
-        <xacro:inertial_cylinder mass="0.1" length="0.0352" radius="0.0206">
-            <origin xyz="0 0 0" rpy="0 0 0"/>
+        <xacro:inertial_cylinder mass="0.1" length="0.0206" radius="0.035">
+            <origin xyz="0 0.115 -0.025" rpy="-${pi/2} 0 0"/>
         </xacro:inertial_cylinder>
     </link>
@@ -125,6 +125,6 @@
             </geometry>
         </collision>
-        <xacro:inertial_cylinder mass="0.1" length="0.0206" radius="0.0352">
-            <origin xyz="0 0 0" rpy="0 0 0"/>
+        <xacro:inertial_cylinder mass="0.1" length="0.0206" radius="0.035">
+            <origin xyz="0 -0.115 -0.025" rpy="${pi/2} 0 0"/>
         </xacro:inertial_cylinder>
     </link>
